File: LEDPanel.kicad_pcb (KiCad board)
At the start: 2 copper layers, 105 x 20 mm, 37 parts, among them J1 Conn_01x08_Pin, J2 Conn_01x02_Pin, Q1 2N3904, Q2 2N3904, Q3 2N3904, Q4 2N3904, Q5 2N3904, Q6 2N3904, Q7 2N3904, Q8 2N3904

Commit message: test commit on test branch
Parts:
- moved REF** 23.3 mm to (144.8, 114.5)

Commit message: test with second sheet
Parts:
- added D9: LED, LED_SMD:LED_0603_1608Metric, F.Cu at (152.5, 127.0)
- moved REF** 23.3 mm to (168.0, 116.2)
Connections:
- net Net-(J2-Pin_1) renamed test4
