File: LEDPanel.kicad_sch (KiCad schematic)
At the start: 34 parts, among them J1 Conn_01x08_Pin, J2 Conn_01x02_Pin, Q1 2N3904, Q2 2N3904, Q3 2N3904, Q4 2N3904, Q5 2N3904, Q6 2N3904, Q7 2N3904, Q8 2N3904

Commit message: test commit on test branch
Other:
- moved on the sheet: Q5
Changed lines of the file:
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@@
+	(wire
+		(pts
+			(xy 189.23 48.26) (xy 144.78 58.42)
+		)
+		(stroke
+			(width 0)
+			(type default)
+		)
+	)
 	(wire
 		(pts
@@
 	(wire
 		(pts
-			(xy 144.78 36.83) (xy 127 36.83)
+			(xy 189.23 36.83) (xy 127 36.83)
+		)
+		(stroke
+			(width 0)
+			(type default)
+		)
+	)
+	(wire
+		(pts
+			(xy 181.61 43.18) (xy 137.16 53.34)
 		)
 		(stroke
@@
 	(wire
 		(pts
-			(xy 144.78 48.26) (xy 144.78 36.83)
+			(xy 189.23 38.1) (xy 189.23 36.83)
 		)
 		(stroke
@@
 	(symbol
 		(lib_id "Transistor_BJT:2N3904")
-		(at 142.24 53.34 0)
+		(at 186.69 43.18 0)
 		(unit 1)
 		(body_style 1)
@@
 		(fields_autoplaced yes)
 		(property "Reference" "Q5"
-			(at 147.32 52.0699 0)
+			(at 191.77 41.9099 0)
 			(show_name no)
 			(do_not_autoplace no)
@@
 		)
 		(property "Value" "2N3904"
-			(at 147.32 54.6099 0)
+			(at 191.77 44.4499 0)
 			(show_name no)
 			(do_not_autoplace no)
@@
 		)
 		(property "Footprint" "Package_TO_SOT_THT:TO-92_HandSolder"
-			(at 147.32 55.245 0)
+			(at 191.77 45.085 0)
 			(hide yes)
 			(show_name no)
@@
 		)
 		(property "Datasheet" "https://www.onsemi.com/pub/Collateral/2N3903-D.PDF"
-			(at 142.24 53.34 0)
+			(at 186.69 43.18 0)
 			(hide yes)
 			(show_name no)
@@
 		)
 		(property "Description" "0.2A Ic, 40V Vce, Small Signal NPN Transistor, TO-92"
-			(at 142.24 53.34 0)
-			(hide yes)
-			(show_name no)
+			(at 186.69 43.18 0)
+			(hide yes)
+			(show_name no)

Commit message: test with second sheet
Connections:
- net global_lable: now reaches J2.1 (Pin_1), Q1.3 (C), Q2.3 (C), Q3.3 (C), Q4.3 (C), Q5.3 (C), Q6.3 (C), Q7.3 (C), Q8.3 (C)
- net label: now reaches Q5.1 (E), R10.1
Other:
- added sheet Test_Sheet (test_sheet.kicad_sch)
Changed lines of the file:
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@@
 	(wire
 		(pts
+			(xy 210.82 76.2) (xy 210.82 81.28)
+		)
+		(stroke
+			(width 0)
+			(type default)
+		)
+	)
+	(wire
+		(pts
 			(xy 148.59 101.6) (xy 152.4 101.6)
 		)
@@
 		)
 	)
+	(label "lable"
+		(at 210.82 76.2 0)
+		(effects
+			(font
+				(size 1.27 1.27)
+			)
+			(justify left bottom)
+		)
+	)
+	(label "label"
+		(at 189.23 48.26 0)
+		(effects
+			(font
+				(size 1.27 1.27)
+			)
+			(justify left bottom)
+		)
+	)
+	(global_label "global_lable"
+		(shape input)
+		(at 189.23 36.83 0)
+		(fields_autoplaced yes)
+		(effects
+			(font
+				(size 1.27 1.27)
+			)
+			(justify left)
+		)
+		(property "Intersheetrefs" "${INTERSHEET_REFS}"
+			(at 203.8262 36.83 0)
+			(hide yes)
+			(show_name no)
+			(do_not_autoplace no)
+			(effects
+				(font
+					(size 1.27 1.27)
+				)
+				(justify left)
+			)
+		)
+	)
 	(symbol
 		(lib_id "Device:R_Small_US")
@@
 				)
 			)
+		)
+	)
+	(sheet
+		(at 196.85 81.28)
+		(size 74.93 43.18)
+		(exclude_from_sim no)
+		(in_bom yes)
+		(on_board yes)
+		(dnp no)
+		(fields_autoplaced yes)
+		(stroke
+			(width 0.1524)
+			(type solid)
+		)
+		(fill
+			(color 0 0 0 0)
+		)
+		(property "Sheetname" "Test_Sheet"
+			(at 196.85 80.5684 0)
+			(show_name no)
+			(do_not_autoplace no)
+			(effects
+				(font
+					(size 1.27 1.27)
+				)
+				(justify left bottom)
+			)
+		)
+		(property "Sheetfile" "test_sheet.kicad_sch"
+			(at 196.85 125.0446 0)
+			(show_name no)
+			(do_not_autoplace no)
+			(effects
+				(font
+					(size 1.27 1.27)
+				)
+				(justify left top)
+			)
+		)
+		(pin "hierarchical_label" input
+			(at 210.82 81.28 90)
+			(effects
+				(font
+					(size 1.27 1.27)
+				)
+				(justify right)
+			)
+		)
+		(instances
+			(project "LEDPanel"
+				(path "/9a3f8280-0d88-4d37-bbab-29e72040df2a"
+					(page "2")
+				)
+			)
